File: KiCad/GR_KS0835F_SLIC_Breakout.kicad_pcb (KiCad board)
At the start: 2 copper layers, 71.7 x 27.7 mm, 25 parts, among them J1 RJ, J2 Conn_01x10, U1 KS0835F

Commit message: Add files via upload
Connections:
- net /~PD renamed /~{PD}
Other:
- net class Default removed
- net class PWR removed
- net class Signals removed
- board text added: "~{PD}"
- board text removed: "~PD"
